Commit message: Remove dummy root

File: urdf/semubot.urdf.xacro (robot description, xacro)
@@ -162,10 +162,3 @@
   <!-- Head -->
   <xacro:head_macro parent="main_body" xyz="0 0 0.705" rpy="0 0 0"/>
-  <!-- Dummy root link -->
-  <link name="dummy_root"/>
-  <joint name="dummy_root_joint" type="fixed">
-    <parent link="dummy_root"/>
-    <child link="base_link"/>
-    <origin xyz="0 0 0" rpy="0 0 0"/>
-  </joint>
 </robot>

Commit message: Adding ros2-control

File: urdf/semubot.urdf.xacro (robot description, xacro)
@@ -162,3 +162,38 @@
   <!-- Head -->
   <xacro:head_macro parent="main_body" xyz="0 0 0.705" rpy="0 0 0"/>
+  <!-- ros2_control Hardware Interface -->
+<ros2_control name="SemubotHardwareSystem" type="system">
+  <hardware>
+    <plugin>semubot_hardware_interface/SemubotHardwareInterface</plugin>
+    <param name="wheel_radius">0.06</param>
+    <param name="base_radius">0.305</param>
+  </hardware>
+  <joint name="omni_ball_1_joint">
+    <command_interface name="velocity">
+      <param name="min">-10.0</param>
+      <param name="max">10.0</param>
+    </command_interface>
+    <state_interface name="position"/>
+    <state_interface name="velocity"/>
+    <state_interface name="effort"/>
+  </joint>
+  <joint name="omni_ball_2_joint">
+    <command_interface name="velocity">
+      <param name="min">-10.0</param>
+      <param name="max">10.0</param>
+    </command_interface>
+    <state_interface name="position"/>
+    <state_interface name="velocity"/>
+    <state_interface name="effort"/>
+  </joint>
+  <joint name="omni_ball_3_joint">
+    <command_interface name="velocity">
+      <param name="min">-10.0</param>
+      <param name="max">10.0</param>
+    </command_interface>
+    <state_interface name="position"/>
+    <state_interface name="velocity"/>
+    <state_interface name="effort"/>
+  </joint>
+</ros2_control>
 </robot>
