Commit message: Make RealSense and ros2_control optional
realsense2_description is only needed with camera:=true, so it is no longer
a package dependency. The ros2_control block moves to a shared macro in
urdf/ros2_control.xacro and is left out with sim:=true, where Gazebo drives
the robot with its own plugins.

File: urdf/semubot.urdf.xacro (robot description, xacro)
@@ -4,4 +4,5 @@
   <xacro:arg name="camera" default="false"/>
   <xacro:include filename="$(find semubot_description)/urdf/head.urdf.xacro"/>
+  <xacro:include filename="$(find semubot_description)/urdf/ros2_control.xacro"/>
   <xacro:if value="$(arg sim)">
     <xacro:include filename="$(find semubot_description)/urdf/semubot.gazebo.xacro"/>
@@ -167,38 +168,7 @@
   <!-- Head -->
   <xacro:head_macro parent="main_body" xyz="0 0 0.705" rpy="0 0 0" sim="$(arg sim)" camera="$(arg camera)"/>
-  <!-- ros2_control Hardware Interface -->
-<ros2_control name="SemubotHardwareSystem" type="system">
-  <hardware>
-    <plugin>semubot_hardware_interface/SemubotHardwareInterface</plugin>
-    <param name="wheel_radius">0.06</param>
-    <param name="base_radius">0.305</param>
-  </hardware>
-  <joint name="omni_ball_1_joint">
-    <command_interface name="velocity">
-      <param name="min">-10.0</param>
-      <param name="max">10.0</param>
-    </command_interface>
-    <state_interface name="position"/>
-    <state_interface name="velocity"/>
-    <state_interface name="effort"/>
-  </joint>
-  <joint name="omni_ball_2_joint">
-    <command_interface name="velocity">
-      <param name="min">-10.0</param>
-      <param name="max">10.0</param>
-    </command_interface>
-    <state_interface name="position"/>
-    <state_interface name="velocity"/>
-    <state_interface name="effort"/>
-  </joint>
-  <joint name="omni_ball_3_joint">
-    <command_interface name="velocity">
-      <param name="min">-10.0</param>
-      <param name="max">10.0</param>
-    </command_interface>
-    <state_interface name="position"/>
-    <state_interface name="velocity"/>
-    <state_interface name="effort"/>
-  </joint>
-</ros2_control>
+  <!-- ros2_control Hardware Interface (real robot only; Gazebo uses its own plugins) -->
+  <xacro:unless value="$(arg sim)">
+    <xacro:semubot_ros2_control wheel_radius="0.06" base_radius="0.305"/>
+  </xacro:unless>
 </robot>
