Commit message: Change mass to SemuBot actual mass

File: urdf/head.urdf.xacro (robot description, xacro)
@@ -18,6 +18,6 @@
       <inertial>
         <origin xyz="0 0 0" rpy="0 0 0"/>
-        <mass value="0.4"/>
-        <inertia ixx="0.01" ixy="0.0" ixz="0.0" iyy="0.01" iyz="0.0" izz="0.01"/>
+        <mass value="1.2"/>
+        <inertia ixx="0.03" ixy="0.0" ixz="0.0" iyy="0.03" iyz="0.0" izz="0.03"/>
       </inertial>
     </link>
@@ -45,6 +45,6 @@
       <inertial>
         <origin xyz="0 0 0" rpy="0 0 0"/>
-        <mass value="0.2"/>
-        <inertia ixx="0.005" ixy="0.0" ixz="0.0" iyy="0.005" iyz="0.0" izz="0.005"/>
+        <mass value="0.6"/>
+        <inertia ixx="0.015" ixy="0.0" ixz="0.0" iyy="0.015" iyz="0.0" izz="0.015"/>
       </inertial>
     </link>
@@ -70,6 +70,6 @@
       <inertial>
         <origin xyz="0 0 0" rpy="0 0 0"/>
-        <mass value="0.2"/>
-        <inertia ixx="0.005" ixy="0.0" ixz="0.0" iyy="0.005" iyz="0.0" izz="0.005"/>
+        <mass value="0.6"/>
+        <inertia ixx="0.015" ixy="0.0" ixz="0.0" iyy="0.015" iyz="0.0" izz="0.015"/>
       </inertial>
     </link>

File: urdf/semubot.urdf.xacro (robot description, xacro)
@@ -28,6 +28,6 @@
     <inertial>
       <origin xyz="0 0 0.02" rpy="0 0 0"/>
-      <mass value="5.0"/>
-      <inertia ixx="0.1" ixy="0.0" ixz="0.0" iyy="0.1" iyz="0.0" izz="0.1"/>
+      <mass value="15.0"/>
+      <inertia ixx="0.3" ixy="0.0" ixz="0.0" iyy="0.3" iyz="0.0" izz="0.3"/>
     </inertial>
   </link>
@@ -56,7 +56,7 @@
   </xacro:macro>
   <!-- Omni-balls -->
-  <xacro:omni_ball_macro name="omni_ball_1" xyz="0 0 0" rpy="0 0 0" scale="1" mass="0.1" ixx="0.001" iyy="0.001" izz="0.001"/>
-  <xacro:omni_ball_macro name="omni_ball_2" xyz="0 0 0" rpy="0 0 0" scale="1" mass="0.1" ixx="0.001" iyy="0.001" izz="0.001"/>
-  <xacro:omni_ball_macro name="omni_ball_3" xyz="0 0 0" rpy="0 0 0" scale="1" mass="0.1" ixx="0.001" iyy="0.001" izz="0.001"/>
+  <xacro:omni_ball_macro name="omni_ball_1" xyz="0 0 0" rpy="0 0 0" scale="1" mass="0.3" ixx="0.003" iyy="0.003" izz="0.003"/>
+  <xacro:omni_ball_macro name="omni_ball_2" xyz="0 0 0" rpy="0 0 0" scale="1" mass="0.3" ixx="0.003" iyy="0.003" izz="0.003"/>
+  <xacro:omni_ball_macro name="omni_ball_3" xyz="0 0 0" rpy="0 0 0" scale="1" mass="0.3" ixx="0.003" iyy="0.003" izz="0.003"/>
   <!-- Joints for Omni-balls -->
   <joint name="omni_ball_1_joint" type="continuous">
@@ -97,6 +97,6 @@
     <inertial>
       <origin xyz="0 0 0.05" rpy="0 0 0"/>
-      <mass value="3.0"/>
-      <inertia ixx="0.05" ixy="0.0" ixz="0.0" iyy="0.05" iyz="0.0" izz="0.05"/>
+      <mass value="9.0"/>
+      <inertia ixx="0.15" ixy="0.0" ixz="0.0" iyy="0.15" iyz="0.0" izz="0.15"/>
     </inertial>
   </link>
@@ -122,6 +122,6 @@
     <inertial>
       <origin xyz="0 0 0" rpy="0 0 0"/>
-      <mass value="0.5"/>
-      <inertia ixx="0.01" ixy="0.0" ixz="0.0" iyy="0.01" iyz="0.0" izz="0.01"/>
+      <mass value="1.5"/>
+      <inertia ixx="0.03" ixy="0.0" ixz="0.0" iyy="0.03" iyz="0.0" izz="0.03"/>
     </inertial>
   </link>
@@ -149,6 +149,6 @@
     <inertial>
       <origin xyz="0 0 0" rpy="0 0 0"/>
-      <mass value="0.5"/>
-      <inertia ixx="0.01" ixy="0.0" ixz="0.0" iyy="0.01" iyz="0.0" izz="0.01"/>
+      <mass value="1.5"/>
+      <inertia ixx="0.03" ixy="0.0" ixz="0.0" iyy="0.03" iyz="0.0" izz="0.03"/>
     </inertial>
   </link>

Commit message: Removed head movement

File: urdf/head.urdf.xacro (robot description, xacro)
@@ -22,10 +22,8 @@
       </inertial>
     </link>
-    <joint name="head_joint" type="revolute">
+    <joint name="head_joint" type="fixed">
       <parent link="${parent}"/>
       <child link="head_base"/>
       <origin xyz="${xyz}" rpy="${rpy}"/>
-      <axis xyz="0 1 0"/>
-      <limit lower="-1.57" upper="1.57" effort="10" velocity="1.0"/>
     </joint>
     <!-- Head Scalp -->

Commit message: Added RealSense D435i compatibility

File: urdf/head.urdf.xacro (robot description, xacro)
@@ -1,5 +1,6 @@
 <?xml version="1.0"?>
 <robot xmlns:xacro="http://www.ros.org/wiki/xacro">
-  <xacro:macro name="head_macro" params="parent xyz rpy">
+  <xacro:include filename="$(find realsense2_description)/urdf/_d435i.urdf.xacro"/>
+  <xacro:macro name="head_macro" params="parent xyz rpy sim:=false">
     <!-- Head Base -->
     <link name="head_base">
@@ -77,4 +78,7 @@
       <origin xyz="0 0 0" rpy="0 0 0"/>
     </joint>
+    <xacro:sensor_d435i parent="head_base" name="camera" use_nominal_extrinsics="${sim}">
+      <origin xyz="0.12 0 0.13" rpy="0 0 0"/>
+    </xacro:sensor_d435i>
   </xacro:macro>
 </robot>

Commit message: Added option to remove camera

File: urdf/head.urdf.xacro (robot description, xacro)
@@ -1,6 +1,8 @@
 <?xml version="1.0"?>
 <robot xmlns:xacro="http://www.ros.org/wiki/xacro">
-  <xacro:include filename="$(find realsense2_description)/urdf/_d435i.urdf.xacro"/>
-  <xacro:macro name="head_macro" params="parent xyz rpy sim:=false">
+  <xacro:if value="$(arg camera)">
+    <xacro:include filename="$(find realsense2_description)/urdf/_d435i.urdf.xacro"/>
+  </xacro:if>
+  <xacro:macro name="head_macro" params="parent xyz rpy sim:=false camera:=false">
     <!-- Head Base -->
     <link name="head_base">
@@ -78,7 +80,9 @@
       <origin xyz="0 0 0" rpy="0 0 0"/>
     </joint>
-    <xacro:sensor_d435i parent="head_base" name="camera" use_nominal_extrinsics="${sim}">
-      <origin xyz="0.12 0 0.13" rpy="0 0 0"/>
-    </xacro:sensor_d435i>
+    <xacro:if value="${camera}">
+      <xacro:sensor_d435i parent="head_base" name="camera" use_nominal_extrinsics="${sim}">
+        <origin xyz="0.12 0 0.13" rpy="0 0 0"/>
+      </xacro:sensor_d435i>
+    </xacro:if>
   </xacro:macro>
 </robot>

File: urdf/semubot.urdf.xacro (robot description, xacro)
@@ -1,6 +1,7 @@
 <?xml version="1.0"?>
 <robot xmlns:xacro="http://www.ros.org/wiki/xacro" name="semubot">
+  <xacro:arg name="sim" default="false"/>
+  <xacro:arg name="camera" default="false"/>
   <xacro:include filename="$(find semubot_description)/urdf/head.urdf.xacro"/>
-  <xacro:arg name="sim" default="false"/>
   <xacro:if value="$(arg sim)">
     <xacro:include filename="$(find semubot_description)/urdf/semubot.gazebo.xacro"/>
@@ -165,5 +166,5 @@
   </joint>
   <!-- Head -->
-  <xacro:head_macro parent="main_body" xyz="0 0 0.705" rpy="0 0 0" sim="$(arg sim)"/>
+  <xacro:head_macro parent="main_body" xyz="0 0 0.705" rpy="0 0 0" sim="$(arg sim)" camera="$(arg camera)"/>
   <!-- ros2_control Hardware Interface -->
 <ros2_control name="SemubotHardwareSystem" type="system">
